File: Hardware/highSide_driver/highSideDriver.sch (KiCad schematic (older format))
At the start: 46 parts

Commit message: PCB design of highside-multiplexer and lowside-switch - New KiCad Lib in Hardware folder
Parts:
- removed C? (x7): CP, symbol CP
- removed C?: C, symbol C
- removed Q? (x8): IRF9310PbF, symbol Q_PMOS_DGS
- removed R? (x8): R, symbol R
- added C1: 100nF, Capacitor_THT:C_Disc_D5.0mm_W2.5mm_P5.00mm, symbol Device:C
- added C10, C11, C5, C6, C7, C8, C9: 10µF, Capacitor_THT:CP_Radial_D7.5mm_P2.50mm, symbol highSideDriver-rescue:CP
- added C12, C2: 33µF, Capacitor_THT:CP_Radial_D13.0mm_P5.00mm, symbol Device:CP
- added C13, C3: 100nF, Capacitor_THT:C_Disc_D11.0mm_W5.0mm_P5.00mm, symbol Device:C
- added J3, J5: Conn_01x02, Connector_Phoenix_MSTB:PhoenixContact_MSTBA_2,5_2-G-5,08_1x02_P5.08mm_Horizontal, symbol Connector_Generic:Conn_01x02
- added Q1, Q2, Q3, Q4, Q5, Q6, Q7, Q8: SI4463, Package_SO:SOIC-8_3.9x4.9mm_P1.27mm, symbol 00_cosi_transistor:SI4463
- C4: renamed from C?; value CP -> 10µF; footprint (none) -> Capacitor_THT:CP_Radial_D7.5mm_P2.50mm; symbol CP -> highSideDriver-rescue:CP
- J1, J2: renamed from J?; footprint (none) -> Connector_IDC:IDC-Header_2x05_P2.54mm_Vertical; symbol Conn_01x10 -> highSideDriver-rescue:Conn_01x10
- J4: renamed from J?; footprint (none) -> Connector_Phoenix_MSTB:PhoenixContact_MSTBA_2,5_8-G-5,08_1x08_P5.08mm_Horizontal; symbol Conn_01x08 -> highSideDriver-rescue:Conn_01x08
- R1, R10, R11, R12, R2, R3, R4, R9: renamed from R?; value R -> 1k; footprint (none) -> Resistor_THT:R_Axial_DIN0204_L3.6mm_D1.6mm_P7.62mm_Horizontal; symbol R -> highSideDriver-rescue:R
- R13, R14, R15, R16, R5, R6, R7, R8: renamed from R?; footprint (none) -> Resistor_SMD:R_0603_1608Metric_Pad0.99x1.00mm_HandSolder; symbol R -> highSideDriver-rescue:R
- R17: renamed from R?; footprint (none) -> Resistor_THT:R_Axial_DIN0204_L3.6mm_D1.6mm_P7.62mm_Horizontal; symbol R -> highSideDriver-rescue:R
- U1: renamed from U?; footprint (none) -> Package_DIP:DIP-16_W7.62mm; symbol TPIC6C595 -> highSideDriver-rescue:TPIC6C595
Connections:
- net labels added: VCC, VDD
- net labels removed: +5V, LED_ANODE_0
- wire segments 137 -> 207
Other:
- note added: "TLC5916ID"
- note added: "Vcc for shift register"
- note added: "Vdd for LEDs"
- moved on the sheet: C4, J1, J2, J4, R1, R10, R11, R12, R17, R2, R3, R4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
