File: Hardware/lowSide_driver/lowSideSwitch.sch (KiCad schematic (older format))
At the start: 32 parts, among them J1 LEDS_0-15, J2 Conn_01x16, J3 Conn_01x16, J4 Conn_01x16, J5 Conn_01x10, J6 Conn_01x10, J7 Conn_01x02, U1 TLC591, U2 TLC591, U3 TLC591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

Commit message: Software: Added timer for LE and OE
Parts:
- added R?: 120, symbol Device:R
- U1, U2, U3, U4, U5, U6, U7, U8: symbol 00_cosi_ic:TLC591 -> lowSideSwitch-rescue:TLC591-00_cosi_ic
Changed lines of the file:
@@
 $EndComp
 $Comp
-L 00_cosi_ic:TLC591 U2
+L lowSideSwitch-rescue:TLC591-00_cosi_ic U2
 U 1 1 5AFEC385
 P 5650 1700
@@
 $EndComp
 $Comp
-L 00_cosi_ic:TLC591 U1
+L lowSideSwitch-rescue:TLC591-00_cosi_ic U1
 U 1 1 5AFEC2CD
 P 3500 1700
@@
 $EndComp
 $Comp
-L 00_cosi_ic:TLC591 U4
+L lowSideSwitch-rescue:TLC591-00_cosi_ic U4
 U 1 1 5B2E821B
 P 9900 1700
@@
 $EndComp
 $Comp
-L 00_cosi_ic:TLC591 U3
+L lowSideSwitch-rescue:TLC591-00_cosi_ic U3
 U 1 1 5B2E8222
 P 7750 1700
@@
 $EndComp
 $Comp
-L 00_cosi_ic:TLC591 U6
+L lowSideSwitch-rescue:TLC591-00_cosi_ic U6
 U 1 1 5B3CA4F6
 P 5650 4200
@@
 $EndComp
 $Comp
-L 00_cosi_ic:TLC591 U5
+L lowSideSwitch-rescue:TLC591-00_cosi_ic U5
 U 1 1 5B3CA4FD
 P 3500 4200
@@
 $EndComp
 $Comp
-L 00_cosi_ic:TLC591 U8
+L lowSideSwitch-rescue:TLC591-00_cosi_ic U8
 U 1 1 5B3CA566
 P 9900 4200
@@
 $EndComp
 $Comp
-L 00_cosi_ic:TLC591 U7
+L lowSideSwitch-rescue:TLC591-00_cosi_ic U7
 U 1 1 5B3CA56D
 P 7750 4200
@@
 NoConn ~ 3500 7100
 NoConn ~ 4700 7100
+$Comp
+L Device:R R?
+U 1 1 5B2F66FC
+P 5300 2700
+F 0 "R?" V 5400 2700 50  0000 C CNN
+F 1 "120" V 5300 2700 50  0000 C CNN
+F 2 "" V 5230 2700 50  0001 C CNN
+F 3 "~" H 5300 2700 50  0001 C CNN
+	1    5300 2700
+	0    -1   -1   0
+$EndComp
 $EndSCHEMATC
